File: PCB/uCschematic.sch (EAGLE design)
At the start: 28 parts, among them IC1 PIC24FJXXGA002/SO, IC10 ULN2003D1013TR, IC11 ULN2003D1013TR, IC12 ULN2003D1013TR, IC2 317EMP, IC3 MC74HC175ADG, IC4 MC74HC175ADG, IC5 MC74HC175ADG, IC6 MC74HC175ADG, IC7 MC74HC175ADG, IC8 MC74HC175ADG, IC9 ULN2003D1013TR, U1 74HC237D-Q100J

Commit message: Made block for each component
Other:
- note added: "MICROCONTROLLER"
- note added: "STEPPER MOTOR CONTROLLER"
- note added: "VOLTAGE REGULATOR"
- moved on the sheet: C4, C5, GND, IC2, R3, R4, U1, VDD

Commit message: Sredjena sema
Parts:
- added GND1, MCLR, PGEC, PGED, RX, SM11, SM12, SM13, SM14, SM21, SM22, SM23, SM24, SM31, SM32, SM33, SM34, SM41, SM42, SM43, SM44, SM51, SM52, SM53, SM54, SM61, SM62, SM63, SM64, TX, VDD_3.3, VDD_PROG, VDD_PROG1, VDD_UC: PIN1-2, con-faston:PIN1-2
- C4, C5: value (none) -> 0.1u
Connections:
- new net N$24: IC1.PGEC2/TMS/PMD1/CN15/RP11/RB11, PGEC.1
- new net N$25: IC1.AN9/PMCS1/CN11/RP15/RB15, RX.1
- new net N$26: IC1.AN10/CVREF/RTCC/PMWR/CN12/RP14/RB14, TX.1
- new net N$27: VDD_PROG.1, VDD_PROG1.1
- net 3.3V: now also VDD_3.3.1
- net GND: now also C3.1, GND1.1, IC1.VSS@0
- net N$2: now also MCLR.1
- net N$30: now also SM11.1
- net N$31: now also SM12.1
- net N$32: now also SM13.1
- net N$33: now also SM14.1
- net N$34: now also SM21.1
- net N$35: now also SM22.1
- net N$36: now also SM23.1
- net N$4: now also VDD_UC.1
- net N$46: now also SM24.1
- net N$47: now also SM31.1
- net N$48: now also SM32.1
- net N$49: now also SM33.1
- net N$50: now also SM34.1
- net N$51: now also SM41.1
- net N$52: now also SM42.1
- net N$62: now also SM43.1
- net N$63: now also SM44.1
- net N$64: now also SM51.1
- net N$65: now also SM52.1
- net N$66: now also SM53.1
- net N$67: now also SM54.1
- net N$68: now also SM61.1
- net N$7: now also IC1.PGED2/TDI/PMD2/CN16/RP10/RB10, PGED.1; no longer C3.1, IC1.VSS@0
- net N$78: now also SM62.1
- net N$79: now also SM63.1
- net N$80: now also SM64.1

Commit message: SPI, I2C, 4 granicna prekidaca, DONE
Parts:
- added CAT_ANGLE, CAT_ROTATION, CS, GP_LASER1, GP_LASER2, MISO, SCLK/SCL, SDA/MOSI: PIN1-2, con-faston:PIN1-2
- added R10, R5, R6, R7, R8, R9: 10k, eagle-ltspice:R
Connections:
- removed net RST: IC1.TCK/SCL1/PMD4/CN22/RP8/RB8, IC3.RESET, IC4.RESET, IC5.RESET, IC6.RESET, IC7.RESET, IC8.RESET
- new net N$29: GP_LASER2.1, IC1.RA1/CN3/VR-/AN1, R6.2
- new net N$37: CAT_ROTATION.1, IC1.RA0/CN2/VR+/AN0, R7.2
- new net N$38: CAT_ANGLE.1, IC1.INT0/PMD5/CN23/RP7/RB7, R8.1
- new net N$39: CS.1, IC1.AN12/PMD0/CN14/RP12/RB12
- new net N$40: IC1.AN11/PMRD/CN13/RP13/RB13, MISO.1
- new net N$41: IC1.AN10/CVREF/RTCC/PMWR/CN12/RP14/RB14, R10.2, SDA/MOSI.1
- new net N$42: IC1.AN9/PMCS1/CN11/RP15/RB15, R9.2, SCLK/SCL.1
- net 3.3V: now also IC3.RESET, IC4.RESET, IC5.RESET, IC6.RESET, IC7.RESET, IC8.RESET, R10.1, R9.1
- net GND: now also R5.1, R6.1, R7.1, R8.2, U1.E2
- net N$17: now also GP_LASER1.1, IC1.RA4/CN0/PMA1/T1CK/SOSCO, R5.2; no longer IC1.INT0/PMD5/CN23/RP7/RB7, U1.E2
- net N$25: now also IC1.TDO/SDA1/PMD3/CN21/RP9/RB9; no longer IC1.AN9/PMCS1/CN11/RP15/RB15
- net N$26: now also IC1.TCK/SCL1/PMD4/CN22/RP8/RB8; no longer IC1.AN10/CVREF/RTCC/PMWR/CN12/RP14/RB14
Other:
- note added: "GP"
- note added: "I2C/SPI"
- note added: "PROGRAMATOR PINS"
- note added: "UART"
- moved on the sheet: GND1, MCLR, PGEC, PGED, RX, TX, VDD_3.3, VDD_PROG, VDD_PROG1, VDD_UC

Commit message: Uradjene izmjene PIN19 spojen na GND Kapacitivnost kondenzatora kod kristala kvarca je sada 47pF Dodana je masa za svaki od GP Dodana je masa za SPI i I2C Dodane su mase za koracne motore LATCH i ENABLE sada su na dobrim logickim nivoima
Parts:
- added GND_CAT_ANGLE, GND_CAT_ROTATION, GND_GP_LASER1, GND_GP_LASER2, GND_SM1, GND_SM2, GND_SM3, GND_SM4, GND_SM5, GND_SM6, GND_SPI/I2C: PIN1-2, con-faston:PIN1-2
- C6, C8: value 100nF -> 47pF
Connections:
- net 3.3V: now also U1.E2
- net GND: now also GND_CAT_ANGLE.1, GND_CAT_ROTATION.1, GND_GP_LASER1.1, GND_GP_LASER2.1, GND_SM1.1, GND_SM2.1, GND_SM3.1, GND_SM4.1, GND_SM5.1, GND_SM6.1, GND_SPI/I2C.1, IC1.DISVREG; no longer U1.E2
Changed lines of the file:
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@@
 <part name="GND" library="con-faston" deviceset="PIN1-2" device=""/>
 <part name="Q1" library="special" library_urn="urn:adsk.eagle:library:367" deviceset="XTAL/S" device="" package3d_urn="urn:adsk.eagle:package:26647/2"/>
-<part name="C6" library="eagle-ltspice" deviceset="C" device="" value="100nF"/>
-<part name="C8" library="eagle-ltspice" deviceset="C" device="" value="100nF"/>
+<part name="C6" library="eagle-ltspice" deviceset="C" device="" value="47pF"/>
+<part name="C8" library="eagle-ltspice" deviceset="C" device="" value="47pF"/>
 <part name="SUPPLY4" library="supply2" deviceset="GND" device=""/>
 <part name="U1" library="74HC237D-Q100J" deviceset="74HC237D-Q100J" device=""/>
@@
 <part name="RX" library="con-faston" deviceset="PIN1-2" device=""/>
 <part name="TX" library="con-faston" deviceset="PIN1-2" device=""/>
-<part name="SUPPLY6" library="supply2" deviceset="GND" device=""/>
 <part name="GP_LASER1" library="con-faston" deviceset="PIN1-2" device=""/>
 <part name="GP_LASER2" library="con-faston" deviceset="PIN1-2" device=""/>
@@
 <part name="R9" library="eagle-ltspice" deviceset="R" device="" value="10k"/>
 <part name="R10" library="eagle-ltspice" deviceset="R" device="" value="10k"/>
+<part name="GND_GP_LASER1" library="con-faston" deviceset="PIN1-2" device=""/>
+<part name="GND_GP_LASER2" library="con-faston" deviceset="PIN1-2" device=""/>
+<part name="GND_CAT_ANGLE" library="con-faston" deviceset="PIN1-2" device=""/>
+<part name="GND_CAT_ROTATION" library="con-faston" deviceset="PIN1-2" device=""/>
+<part name="GND_SPI/I2C" library="con-faston" deviceset="PIN1-2" device=""/>
+<part name="GND_SM1" library="con-faston" deviceset="PIN1-2" device=""/>
+<part name="GND_SM2" library="con-faston" deviceset="PIN1-2" device=""/>
+<part name="GND_SM3" library="con-faston" deviceset="PIN1-2" device=""/>
+<part name="GND_SM4" library="con-faston" deviceset="PIN1-2" device=""/>
+<part name="GND_SM5" library="con-faston" deviceset="PIN1-2" device=""/>
+<part name="GND_SM6" library="con-faston" deviceset="PIN1-2" device=""/>
 </parts>
 <sheets>
@@
 <text x="165.1" y="-124.46" size="1.778" layer="91">UART</text>
 <text x="213.36" y="-124.46" size="1.778" layer="91">I2C/SPI</text>
-<text x="127" y="177.8" size="1.778" layer="91">GP</text>
+<text x="154.94" y="177.8" size="1.778" layer="91">GP</text>
 </plain>
 <instances>
@@
 <attribute name="NAME" x="161.29" y="-104.14" size="1.778" layer="95" rot="R270"/>
 </instance>
-<instance part="SUPPLY6" gate="GND" x="220.98" y="30.48" smashed="yes" rot="R270">
-<attribute name="VALUE" x="217.805" y="32.385" size="1.778" layer="96" rot="R270"/>
-</instance>
 <instance part="GP_LASER1" gate="G$1" x="86.36" y="193.04" smashed="yes" rot="R90">
 <attribute name="NAME" x="85.09" y="190.5" size="1.778" layer="95" rot="R90"/>
@@
 <attribute name="NAME" x="189.23" y="-59.4614" size="1.778" layer="95"/>
 <attribute name="VALUE" x="189.23" y="-64.262" size="1.778" layer="96"/>
+</instance>
+<instance part="GND_GP_LASER1" gate="G$1" x="116.84" y="193.04" smashed="yes" rot="R90">
+<attribute name="NAME" x="115.57" y="190.5" size="1.778" layer="95" rot="R90"/>
+</instance>
+<instance part="GND_GP_LASER2" gate="G$1" x="124.46" y="193.04" smashed="yes" rot="R90">
+<attribute name="NAME" x="123.19" y="190.5" size="1.778" layer="95" rot="R90"/>
+</instance>
+<instance part="GND_CAT_ANGLE" gate="G$1" x="139.7" y="193.04" smashed="yes" rot="R90">
+<attribute name="NAME" x="138.43" y="190.5" size="1.778" layer="95" rot="R90"/>
+</instance>
+<instance part="GND_CAT_ROTATION" gate="G$1" x="132.08" y="193.04" smashed="yes" rot="R90">
+<attribute name="NAME" x="130.81" y="190.5" size="1.778" layer="95" rot="R90"/>
+</instance>
+<instance part="GND_SPI/I2C" gate="G$1" x="187.96" y="-114.3" smashed="yes" rot="R270">
+<attribute name="NAME" x="189.23" y="-111.76" size="1.778" layer="95" rot="R270"/>
+</instance>
+<instance part="GND_SM1" gate="G$1" x="474.98" y="-10.16" smashed="yes">
+<attribute name="NAME" x="472.44" y="-11.43" size="1.778" layer="95"/>
+</instance>
+<instance part="GND_SM2" gate="G$1" x="474.98" y="-15.24" smashed="yes">
+<attribute name="NAME" x="472.44" y="-16.51" size="1.778" layer="95"/>
+</instance>
+<instance part="GND_SM3" gate="G$1" x="474.98" y="-20.32" smashed="yes">
+<attribute name="NAME" x="472.44" y="-21.59" size="1.778" layer="95"/>
+</instance>
+<instance part="GND_SM4" gate="G$1" x="474.98" y="-25.4" smashed="yes">
+<attribute name="NAME" x="472.44" y="-26.67" size="1.778" layer="95"/>
+</instance>
+<instance part="GND_SM5" gate="G$1" x="474.98" y="-30.48" smashed="yes">
+<attribute name="NAME" x="472.44" y="-31.75" size="1.778" layer="95"/>
+</instance>
+<instance part="GND_SM6" gate="G$1" x="474.98" y="-35.56" smashed="yes">
+<attribute name="NAME" x="472.44" y="-36.83" size="1.778" layer="95"/>
 </instance>
 </instances>
@@
 </segment>
 <segment>
-<pinref part="U1" gate="G$1" pin="E2"/>
-<pinref part="SUPPLY6" gate="GND" pin="GND"/>
-<wire x1="236.22" y1="30.48" x2="223.52" y2="30.48" width="0.1524" layer="91"/>
-</segment>
-<segment>
 <pinref part="R7" gate="G$1" pin="1"/>
 <wire x1="114.3" y1="152.4" x2="134.62" y2="152.4" width="0.1524" layer="91"/>
@@
 <wire x1="134.62" y1="160.02" x2="144.78" y2="160.02" width="0.1524" layer="91"/>
 <wire x1="144.78" y1="160.02" x2="144.78" y2="165.1" width="0.1524" layer="91"/>
+<pinref part="GND_GP_LASER1" gate="G$1" pin="1"/>
+<wire x1="116.84" y1="187.96" x2="116.84" y2="185.42" width="0.1524" layer="91"/>
+<wire x1="116.84" y1="185.42" x2="124.46" y2="185.42" width="0.1524" layer="91"/>
+<pinref part="GND_CAT_ANGLE" gate="G$1" pin="1"/>
+<wire x1="124.46" y1="185.42" x2="132.08" y2="185.42" width="0.1524" layer="91"/>
+<wire x1="132.08" y1="185.42" x2="134.62" y2="185.42" width="0.1524" layer="91"/>
+<wire x1="134.62" y1="185.42" x2="139.7" y2="185.42" width="0.1524" layer="91"/>
+<wire x1="139.7" y1="185.42" x2="139.7" y2="187.96" width="0.1524" layer="91"/>
+<pinref part="GND_CAT_ROTATION" gate="G$1" pin="1"/>
+<wire x1="132.08" y1="187.96" x2="132.08" y2="185.42" width="0.1524" layer="91"/>
+<junction x="132.08" y="185.42"/>
+<pinref part="GND_GP_LASER2" gate="G$1" pin="1"/>
+<wire x1="124.46" y1="187.96" x2="124.46" y2="185.42" width="0.1524" layer="91"/>
+<junction x="124.46" y="185.42"/>
+<wire x1="134.62" y1="185.42" x2="134.62" y2="167.64" width="0.1524" layer="91"/>
+<junction x="134.62" y="185.42"/>
+<junction x="134.62" y="167.64"/>
+</segment>
+<segment>
+<pinref part="GND_SPI/I2C" gate="G$1" pin="1"/>
+<wire x1="187.96" y1="-109.22" x2="187.96" y2="-106.68" width="0.1524" layer="91"/>
+<label x="187.96" y="-106.68" size="1.778" layer="95" rot="R90" xref="yes"/>
+</segment>
+<segment>
+<pinref part="GND_SM1" gate="G$1" pin="1"/>
+<wire x1="469.9" y1="-10.16" x2="467.36" y2="-10.16" width="0.1524" layer="91"/>
+<pinref part="GND_SM2" gate="G$1" pin="1"/>
+<wire x1="469.9" y1="-15.24" x2="467.36" y2="-15.24" width="0.1524" layer="91"/>
+<wire x1="467.36" y1="-10.16" x2="467.36" y2="-15.24" width="0.1524" layer="91"/>
+<pinref part="GND_SM3" gate="G$1" pin="1"/>
+<wire x1="469.9" y1="-20.32" x2="467.36" y2="-20.32" width="0.1524" layer="91"/>
+<wire x1="467.36" y1="-15.24" x2="467.36" y2="-20.32" width="0.1524" layer="91"/>
+<junction x="467.36" y="-15.24"/>
+<pinref part="GND_SM4" gate="G$1" pin="1"/>
+<wire x1="469.9" y1="-25.4" x2="467.36" y2="-25.4" width="0.1524" layer="91"/>
+<wire x1="467.36" y1="-20.32" x2="467.36" y2="-25.4" width="0.1524" layer="91"/>
+<junction x="467.36" y="-20.32"/>
+<pinref part="GND_SM5" gate="G$1" pin="1"/>
+<wire x1="469.9" y1="-30.48" x2="467.36" y2="-30.48" width="0.1524" layer="91"/>
+<wire x1="467.36" y1="-25.4" x2="467.36" y2="-30.48" width="0.1524" layer="91"/>
+<junction x="467.36" y="-25.4"/>
+<pinref part="GND_SM6" gate="G$1" pin="1"/>
+<wire x1="469.9" y1="-35.56" x2="467.36" y2="-35.56" width="0.1524" layer="91"/>
+<wire x1="467.36" y1="-30.48" x2="467.36" y2="-35.56" width="0.1524" layer="91"/>
+<junction x="467.36" y="-30.48"/>
+<label x="467.36" y="-20.32" size="1.778" layer="95" rot="R180" xref="yes"/>
+</segment>
+<segment>
+<pinref part="IC1" gate="G$1" pin="DISVREG"/>
+<wire x1="96.52" y1="50.8" x2="93.98" y2="50.8" width="0.1524" layer="91"/>
+<label x="93.98" y="50.8" size="1.778" layer="95" rot="R90" xref="yes"/>
 </segment>
 </net>
@@
 <junction x="182.88" y="-63.5"/>
 <label x="180.34" y="-63.5" size="1.778" layer="95" rot="R180" xref="yes"/>
+</segment>
+<segment>
+<pinref part="U1" gate="G$1" pin="E2"/>
+<wire x1="236.22" y1="30.48" x2="233.68" y2="30.48" width="0.1524" layer="91"/>
+<label x="233.68" y="30.48" size="1.778" layer="95" rot="R180" xref="yes"/>
 </segment>
 </net>
@@
 <segment>
 <wire x1="68.58" y1="213.36" x2="68.58" y2="175.26" width="0.1524" layer="91"/>
-<wire x1="68.58" y1="175.26" x2="132.08" y2="175.26" width="0.1524" layer="91"/>
-<wire x1="132.08" y1="175.26" x2="132.08" y2="213.36" width="0.1524" layer="91"/>
-<wire x1="132.08" y1="213.36" x2="68.58" y2="213.36" width="0.1524" layer="91"/>
-</segment>
-</net>
+<wire x1="68.58" y1="175.26" x2="160.02" y2="175.26" width="0.1524" layer="91"/>
+<wire x1="160.02" y1="175.26" x2="160.02" y2="213.36" width="0.1524" layer="91"/>
+<wire x1="160.02" y1="213.36" x2="68.58" y2="213.36" width="0.1524" layer="91"/>
+</segment>
+</net>

Commit message: Uradjena sema za USB/UART converter
Parts:
- removed RX, TX: PIN1-2, con-faston:PIN1-2
- added C10, C11: 47pF, eagle-ltspice:C
- added C9: 0.1u, eagle-ltspice:C
- added IC13: FT230XS-U, FT230XS-U:FT230XS-U
- added J1: USB3075-30-A, USB3075-30-A:USB3075-30-A
- added R11, R12: 27, rcl:R-EU_R0805
Connections:
- new net N$45: C10.2, J1.2, R11.2
- new net N$53: C9.2, IC13.3V3OUT, IC13.RESET#, IC13.VCCIO
- new net N$54: C11.2, J1.3, R12.2
- new net N$55: IC13.USBDM, R11.1
- new net N$56: IC13.USBDP, R12.1
- net 3.3V: now also IC13.VCC
- net GND: now also C10.1, C11.1, C9.1, IC13.GND_1, IC13.GND_2, J1.5, J1.MH1, J1.MH2, J1.MP1, J1.MP2, J1.MP3, J1.MP4
- net N$25: now also IC13.RXD; no longer RX.1
- net N$26: now also IC13.TXD; no longer TX.1
Other:
- note added: "Mozda treba softverski rijesiti pinove za TX i RX"
- note added: "USB/UART converter"
- note removed: "UART"

Commit message: -Dodani bajpas kondenzatori.
Parts:
- added C12, C13, C14, C15, C16, C17, C18, C19, C20, C21, C22, C23, C24, C25, C26: 0.1u, capacitor-wima:C2,5-3
- C4: value 0.1u -> 1u
- R3: value 470 -> 240
- R4: value 770,8 -> 390
Connections:
- new net N$28: C24.2
- new net N$58: C25.2
- new net N$59: C23.2
- new net N$60: C26.2
- new net N$61: C22.2
- new net N$69: C21.2
- new net N$70: C19.2
- new net N$71: C20.2
- new net N$72: C18.2
- new net N$77: C17.2
- new net N$85: C15.2
- net 3.3V: now also C12.1, C13.1, C14.1, C15.1, C16.1, C17.1, C18.1, C19.1, C20.1, C21.1, C22.1, C23.1, C24.1, C25.1, C26.1
- net GND: now also C12.2, C13.2, C14.2, C16.2

Commit message: -Unesene potrebne izmjene
Parts:
- removed C13, C16, C18, C20, C22, C24, C26: 0.1u, capacitor-wima:C2,5-3
Connections:
- removed net N$28: C24.2
- removed net N$60: C26.2
- removed net N$61: C22.2
- removed net N$71: C20.2
- removed net N$72: C18.2
- net 3.3V: no longer C13.1, C16.1, C18.1, C20.1, C22.1, C24.1, C26.1
- net GND: no longer C13.2, C16.2

Commit message: Osiguravanje dodatnog GP u slucaju da bude potreban.
Parts:
- removed C21, C23, C25: 0.1u, capacitor-wima:C2,5-3
- added C13, C16, C18: 0.1u, eagle-ltspice:C
- added GND_GP_1, GP, GP_1, PGEC/GP, PGEC_PROG: PIN1-2, con-faston:PIN1-2
- C12, C14, C15, C17, C19: device capacitor-wima:C2,5-3 -> eagle-ltspice:C
Connections:
- new net GP_1: GP.1, GP_1.1
- new net N$28: PGEC.1, PGEC_PROG.1
- net 3.3V: now also C12.2, C13.2, C14.2, C15.2, C16.2, C17.2, C18.2, C19.2; no longer C12.1, C14.1, C15.1, C17.1, C19.1, C21.1, C23.1, C25.1
- net GND: now also C12.1, C14.1, GND_GP_1.1; no longer C12.2, C14.2
- net N$24: now also PGEC/GP.1; no longer PGEC.1
- net N$58: now also C19.1; no longer C25.2
- net N$59: now also C18.1; no longer C23.2
- net N$69: now also C17.1; no longer C21.2
- net N$70: now also C16.1; no longer C19.2
- net N$77: now also C13.1; no longer C17.2
- net N$85: now also C15.1; no longer C15.2
Other:
- moved on the sheet: C12, C14, C15, C17, C19
