File: PCB/uCschematic.sch (EAGLE design)
At the start: 105 parts, among them IC1 PIC24FJXXGA002/SO, IC10 ULN2003D1013TR, IC11 ULN2003D1013TR, IC12 ULN2003D1013TR, IC13 FT230XS-U, IC2 317EMP, IC3 MC74HC175ADG, IC4 MC74HC175ADG, IC5 MC74HC175ADG, IC6 MC74HC175ADG, IC7 MC74HC175ADG, IC8 MC74HC175ADG, IC9 ULN2003D1013TR, J1 USB3075-30-A, U1 74HC237D-Q100J

Commit message: Uradjena simulacija u proteusu USB micro AB -> USB type A Izvrsena simulacija u proteusu. Sve radi kako treba Izvrsene sitne izmjene na semi
Parts:
- removed GND_GP_1, GP_1: PIN1-2, con-faston:PIN1-2
- removed J1: USB3075-30-A, USB3075-30-A:USB3075-30-A
- added GND_GP_OKIDAC, GP_OKIDAC: PIN1-2, con-faston:PIN1-2
- added J2: USB1046-GF-0190-L-B-A, USB1046-GF-0190-L-B-A:USB1046-GF-0190-L-B-A
- added R13: 10k, eagle-ltspice:R
- renumbered GND_SM1 to 12V_SM1, GND_SM2 to 12V_SM2, GND_SM3 to 12V_SM3, GND_SM4 to 12V_SM4, GND_SM5 to 12V_SM5, GND_SM6 to 12V_SM6
Connections:
- removed net GP_1: GP.1, GP_1.1
- removed net VDD: C5.2, IC10.COMMON_FREE_WHEELING_DIODES, IC11.COMMON_FREE_WHEELING_DIODES, IC12.COMMON_FREE_WHEELING_DIODES, IC2.VI, IC9.COMMON_FREE_WHEELING_DIODES, VDD.1
- new net 12V: 12V_SM1.1, 12V_SM2.1, 12V_SM3.1, 12V_SM4.1, 12V_SM5.1, 12V_SM6.1, C5.2, IC10.COMMON_FREE_WHEELING_DIODES, IC11.COMMON_FREE_WHEELING_DIODES, IC12.COMMON_FREE_WHEELING_DIODES, IC2.VI, IC9.COMMON_FREE_WHEELING_DIODES, VDD.1
- new net GP_OKIDAC: GP.1, GP_OKIDAC.1, R13.2
- net 3.3V: now also R13.1, R5.1, R6.1, R7.1, R8.2
- net GND: now also GND_GP_OKIDAC.1, J2.4, J2.MH1, J2.MH2; no longer 12V_SM1.1, 12V_SM2.1, 12V_SM3.1, 12V_SM4.1, 12V_SM5.1, 12V_SM6.1, GND_GP_1.1, J1.5, J1.MH1, J1.MH2, J1.MP1, J1.MP2, J1.MP3, J1.MP4, R5.1, R6.1, R7.1, R8.2
- net N$45: now also J2.2; no longer J1.2
- net N$54: now also J2.3; no longer J1.3
Other:
- moved on the sheet: CAT_ANGLE, CAT_ROTATION, GND_CAT_ANGLE, GND_CAT_ROTATION, GND_GP_LASER1, GND_GP_LASER2, GP_LASER1, GP_LASER2
